File: layouts/Nose/Nose.kicad_pcb (KiCad board)
At the start: 2 copper layers, 3 parts

Commit message: maintainence
Connections:
- net VDD renamed VDDIO
Changed lines of the file:
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@@
     )
     (net 0 "")
-    (net 1 "VDD")
+    (net 1 "VDDIO")
     (net 2 "SDO")
     (net 3 "SCK")
@@
             (size 0.45 0.89)
             (layers "F.Cu" "F.Mask" "F.Paste")
-            (net 1 "VDD")
+            (net 1 "VDDIO")
         )
         (pad "7" smd rect
@@
             (size 0.45 0.89)
             (layers "F.Cu" "F.Mask" "F.Paste")
-            (net 1 "VDD")
+            (net 1 "VDDIO")
         )
         (embedded_fonts no)
@@
             (size 0.79 0.54)
             (layers "F.Cu" "F.Mask" "F.Paste")
-            (net 1 "VDD")
+            (net 1 "VDDIO")
         )
         (pad "2" smd rect
@@
             (size 0.79 0.54)
             (layers "F.Cu" "F.Mask" "F.Paste")
-            (net 1 "VDD")
+            (net 1 "VDDIO")
         )
         (pad "2" smd rect

Commit message: meow
Connections:
- net VDDIO renamed VDD
Changed lines of the file:
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@@
     )
     (net 0 "")
-    (net 1 "VDDIO")
+    (net 1 "VDD")
     (net 2 "SDO")
     (net 3 "SCK")
@@
             (size 0.45 0.89)
             (layers "F.Cu" "F.Mask" "F.Paste")
-            (net 1 "VDDIO")
+            (net 1 "VDD")
         )
         (pad "7" smd rect
@@
             (size 0.45 0.89)
             (layers "F.Cu" "F.Mask" "F.Paste")
-            (net 1 "VDDIO")
+            (net 1 "VDD")
         )
         (embedded_fonts no)
@@
             (size 0.79 0.54)
             (layers "F.Cu" "F.Mask" "F.Paste")
-            (net 1 "VDDIO")
+            (net 1 "VDD")
         )
         (pad "2" smd rect
@@
             (size 0.79 0.54)
             (layers "F.Cu" "F.Mask" "F.Paste")
-            (net 1 "VDDIO")
+            (net 1 "VDD")
         )
         (pad "2" smd rect
