File: layouts/NoseI2C/NoseI2C.kicad_pcb (KiCad board)
At the start: 2 copper layers, 5 parts

Commit message: doneish
Connections:
- net VDDIO renamed CSB
Changed lines of the file:
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@@
     (net 2 "SDI")
     (net 3 "SDO")
-    (net 4 "VDDIO")
+    (net 4 "CSB")
     (net 5 "gnd")
     (footprint "atopile:R0402-56259e"
@@
             (size 0.57 0.54)
             (layers "F.Cu" "F.Mask" "F.Paste")
-            (net 4 "VDDIO")
+            (net 4 "CSB")
         )
         (embedded_fonts no)
@@
             (size 0.79 0.54)
             (layers "F.Cu" "F.Mask" "F.Paste")
-            (net 4 "VDDIO")
+            (net 4 "CSB")
         )
         (pad "2" smd rect
@@
             (size 0.79 0.54)
             (layers "F.Cu" "F.Mask" "F.Paste")
-            (net 4 "VDDIO")
+            (net 4 "CSB")
         )
         (pad "2" smd rect
@@
             (size 0.45 0.89)
             (layers "F.Cu" "F.Mask" "F.Paste")
-            (net 4 "VDDIO")
+            (net 4 "CSB")
         )
         (pad "3" smd rect
@@
             (size 0.45 0.89)
             (layers "F.Cu" "F.Mask" "F.Paste")
-            (net 4 "VDDIO")
+            (net 4 "CSB")
         )
         (pad "7" smd rect
@@
             (size 0.45 0.89)
             (layers "F.Cu" "F.Mask" "F.Paste")
-            (net 4 "VDDIO")
+            (net 4 "CSB")
         )
         (embedded_fonts no)
@@
             (size 0.57 0.54)
             (layers "F.Cu" "F.Mask" "F.Paste")
-            (net 4 "VDDIO")
+            (net 4 "CSB")
         )
         (embedded_fonts no)

Commit message: meow
Parts:
- R1, R2: value 1kΩ ±1% 62.5mW -> 10kΩ ±1% 62.5mW
Connections:
- net CSB renamed VDDIO
Changed lines of the file:
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@@
     (net 2 "SDI")
     (net 3 "SDO")
-    (net 4 "CSB")
+    (net 4 "VDDIO")
     (net 5 "gnd")
     (footprint "atopile:R0402-56259e"
@@
             )
         )
-        (property "Value" "1kΩ ±1% 62.5mW"
+        (property "Value" "10kΩ ±1% 62.5mW"
             (at 0 0 90)
             (layer "F.Fab")
@@
             )
         )
-        (property "LCSC" "C11702"
-            (at 0 0 90)
-            (layer "User.9")
-            (hide yes)
-            (effects
-                (font
-                    (size 0.125 0.125)
-                    (thickness 0.01875)
-                )
-            )
-        )
-        (property "Partnumber" "0402WGF1001TCE"
+        (property "LCSC" "C25744"
+            (at 0 0 90)
+            (layer "User.9")
+            (hide yes)
+            (effects
+                (font
+                    (size 0.125 0.125)
+                    (thickness 0.01875)
+                )
+            )
+        )
+        (property "Partnumber" "0402WGF1002TCE"
             (at 0 0 90)
             (layer "User.9")
@@
             )
         )
-        (property "JLCPCB description" "62.5mW Thick Film Resistors 50V ±100ppm/℃ ±1% 1kΩ 0402 Chip Resistor - Surface Mount ROHS"
+        (property "JLCPCB description" "62.5mW Thick Film Resistors 50V ±100ppm/℃ ±1% 10kΩ 0402 Chip Resistor - Surface Mount ROHS"
             (at 0 0 90)
             (layer "User.9")
@@
             )
         )
-        (property "PARAM_resistance" "{\"type\": \"Quantity_Interval_Disjoint\", \"data\": {\"intervals\": {\"type\": \"Numeric_Interval_Disjoint\", \"data\": {\"intervals\": [{\"type\": \"Numeric_Interval\", \"data\": {\"min\": 990.0000002235174, \"max\": 1009.9999997764826}}]}}, \"unit\": \"ohm\"}}"
+        (property "PARAM_resistance" "{\"type\": \"Quantity_Interval_Disjoint\", \"data\": {\"intervals\": {\"type\": \"Numeric_Interval_Disjoint\", \"data\": {\"intervals\": [{\"type\": \"Numeric_Interval\", \"data\": {\"min\": 9900.000002235174, \"max\": 10099.999997764826}}]}}, \"unit\": \"ohm\"}}"
             (at 0 0 90)
             (layer "User.9")
@@
             (size 0.57 0.54)
             (layers "F.Cu" "F.Mask" "F.Paste")
-            (net 4 "CSB")
+            (net 4 "VDDIO")
         )
         (embedded_fonts no)
@@
             (size 0.79 0.54)
             (layers "F.Cu" "F.Mask" "F.Paste")
-            (net 4 "CSB")
+            (net 4 "VDDIO")
         )
         (pad "2" smd rect
@@
             (size 0.79 0.54)
             (layers "F.Cu" "F.Mask" "F.Paste")
-            (net 4 "CSB")
+            (net 4 "VDDIO")
         )
         (pad "2" smd rect
@@
             (size 0.45 0.89)
             (layers "F.Cu" "F.Mask" "F.Paste")
-            (net 4 "CSB")
+            (net 4 "VDDIO")
         )
         (pad "3" smd rect
@@
             (size 0.45 0.89)
             (layers "F.Cu" "F.Mask" "F.Paste")
-            (net 4 "CSB")
+            (net 4 "VDDIO")
         )
         (pad "7" smd rect
@@
             (size 0.45 0.89)
             (layers "F.Cu" "F.Mask" "F.Paste")
-            (net 4 "CSB")
+            (net 4 "VDDIO")
         )
         (embedded_fonts no)
@@
             )
         )
-        (property "Value" "1kΩ ±1% 62.5mW"
+        (property "Value" "10kΩ ±1% 62.5mW"
             (at 0 0 90)
             (layer "F.Fab")
@@
             )
         )
-        (property "LCSC" "C11702"
-            (at 0 0 90)
-            (layer "User.9")
-            (hide yes)
-            (effects
-                (font
-                    (size 0.125 0.125)
-                    (thickness 0.01875)
-                )
-            )
-        )
-        (property "Partnumber" "0402WGF1001TCE"
+        (property "LCSC" "C25744"
+            (at 0 0 90)
+            (layer "User.9")
+            (hide yes)
+            (effects
+                (font
+                    (size 0.125 0.125)
+                    (thickness 0.01875)
+                )
+            )
+        )
+        (property "Partnumber" "0402WGF1002TCE"
             (at 0 0 90)
             (layer "User.9")
@@
             )
         )
-        (property "JLCPCB description" "62.5mW Thick Film Resistors 50V ±100ppm/℃ ±1% 1kΩ 0402 Chip Resistor - Surface Mount ROHS"
+        (property "JLCPCB description" "62.5mW Thick Film Resistors 50V ±100ppm/℃ ±1% 10kΩ 0402 Chip Resistor - Surface Mount ROHS"
             (at 0 0 90)
             (layer "User.9")
@@
             )
         )
-        (property "PARAM_resistance" "{\"type\": \"Quantity_Interval_Disjoint\", \"data\": {\"intervals\": {\"type\": \"Numeric_Interval_Disjoint\", \"data\": {\"intervals\": [{\"type\": \"Numeric_Interval\", \"data\": {\"min\": 990.0000002235174, \"max\": 1009.9999997764826}}]}}, \"unit\": \"ohm\"}}"
+        (property "PARAM_resistance" "{\"type\": \"Quantity_Interval_Disjoint\", \"data\": {\"intervals\": {\"type\": \"Numeric_Interval_Disjoint\", \"data\": {\"intervals\": [{\"type\": \"Numeric_Interval\", \"data\": {\"min\": 9900.000002235174, \"max\": 10099.999997764826}}]}}, \"unit\": \"ohm\"}}"
             (at 0 0 90)
             (layer "User.9")
@@
             (size 0.57 0.54)
             (layers "F.Cu" "F.Mask" "F.Paste")
-            (net 4 "CSB")
+            (net 4 "VDDIO")
         )
         (embedded_fonts no)
