File: layouts/nose/nose.kicad_pcb (KiCad board)
At the start: 2 copper layers, 5 parts

Commit message: more
Parts:
- removed R1, R2: 10kΩ ±1% 62.5mW, atopile:R0402-56259e
- moved C2 136.4 mm to (126.8, 98.3), turned to 180 degrees
- moved C1 136.2 mm to (126.8, 100.0), turned to 180 degrees
- moved U1 135.7 mm to (130.1, 99.6)
Connections:
- C1 pad 1: VDD -> VDDIO
- C2 pad 1: VDD -> VDDIO
- U1 pad 2: VDDIO -> CSB
- U1 pad 8: VDD -> VDDIO
Routing:
- net gnd: track 6.29 -> 2.69 mm, vias 0 -> 4
- net VDDIO: track 6.18 -> 2.71 mm
- net VDD: track 3.16 -> 0.00 mm
- net SCK: track 2.68 -> 0.00 mm
- net SDI: track 1.49 -> 0.00 mm
